File: svxlink_interface.kicad_sch (KiCad schematic)
At the start: 16 parts, among them J1 MTM5400 acc.con., J2 RCJ-2123, J3 RPi-GPIO xx, J5 FTDI USB>UART, T1-RX1 600ohm 1:1, T2-TX1 600ohm 1:1, U1 CNY17-2

Commit message: Add files via upload
Parts:
- added D1, D2, D3: 1.5KE6.8CA, Diode_THT:D_DO-201AE_P15.24mm_Horizontal, symbol Diode:1.5KExxCA
Connections:
- net CTS: now also D3.2 (A2)
- net GND: now also D1.1 (A1), D2.1 (A1), D3.1 (A1)
- net RXD: now also D1.2 (A2)
- net TXD: now also D2.2 (A2)
