File: svxlink_interface.kicad_pcb (KiCad board)
At the start: 2 copper layers, 17 parts, among them J1 MTM5400 acc.con., J2 RCJ-2123, J3 RPi-GPIO xx, J5 FTDI USB>UART, T1-RX1 600ohm 1:1, T2-TX1 600ohm 1:1, U1 CNY17-2

Commit message: Add files via upload
Parts:
- added D1: 1.5KE6.8CA, Diode_THT:D_DO-201AE_P15.24mm_Horizontal, F.Cu at (49.8, 34.0)
- added D2: 1.5KE6.8CA, Diode_THT:D_DO-201AE_P15.24mm_Horizontal, F.Cu at (49.8, 41.0)
- added D3: 1.5KE6.8CA, Diode_THT:D_DO-201AE_P15.24mm_Horizontal, F.Cu at (49.8, 48.0)
Connections:
- net Net-(J2-Pad1) renamed GNDS
Routing:
- net RXD: track 44.8 -> 50.9 mm
- net TXD: track 48.9 -> 54.1 mm
- net CTS: track 36.4 -> 41.1 mm

Commit message: Add files via upload
Parts:
- moved J5 6.35 mm to (76.3, 48.0)
- moved D1 5.37 mm to (55.1, 34.0)
- moved D2 5.37 mm to (55.1, 41.0)
- moved D3 5.37 mm to (55.1, 48.0)
- moved C1 4.78 mm to (127.8, 59.0)
- moved R1 4.22 mm to (122.2, 69.8)
- moved R4 2.26 mm to (122.2, 92.8)
Routing:
- net RXD: track 50.9 -> 64.4 mm
- net GND: track 0.00 -> 12.0 mm, vias 0 -> 16
- net GND_MIC: track 57.7 -> 66.6 mm, vias 0 -> 2
- net TXD: track 54.1 -> 45.4 mm
- net Net-(J1-PTT): track 36.2 -> 28.2 mm, vias 0 -> 2
- net CTS: track 41.1 -> 34.2 mm
- net Net-(J2-Pad2): track 10.7 -> 7.97 mm
- net Net-(C1-Pad2): track 12.5 -> 10.5 mm
- net Net-(JP1-C): track 37.8 -> 35.9 mm
- net Net-(R1-Pad1): track 9.25 -> 10.3 mm
- net Net-(C1-Pad1): track 4.87 -> 5.92 mm
- net Net-(R4-Pad1): track 9.63 -> 10.3 mm
- net Net-(J1-EXT_MIC): vias 0 -> 2
Other:
- board text added: "FTDI USB - UART converter"
- board text added: "Isolated SVXLink interface from usb-audio card to MTM5400"
- board text added: "v1.4"
- board text removed: "FTDI USB to Serial (UART) convertor"
- board text removed: "Isolated SVXLink-RPi modem from CM108 to MTM5400"

Commit message: Add files via upload
Parts:
- moved J5 9.65 mm to (84.9, 52.4)
- moved D1 9.65 mm to (63.7, 38.4)
- moved D2 9.65 mm to (63.7, 45.4)
- moved D3 9.62 mm to (63.8, 52.2)
- moved J3 7.25 mm to (75.0, 107.1)
- moved R5 7.25 mm to (81.3, 107.1)
- moved R6 7.25 mm to (66.8, 102.1)
- moved U1 7.25 mm to (69.0, 97.8)
- moved REF** 1.82 mm to (128.5, 103.2)
Routing:
- net TXD: track 45.4 -> 67.8 mm
- net RXD: track 64.4 -> 80.3 mm
- net Net-(J1-PTT): track 28.2 -> 35.9 mm
- net CTS: track 34.2 -> 41.4 mm
- net GND_MIC: track 66.6 -> 63.1 mm
- net Net-(J1-RX_Audio): track 46.3 -> 45.1 mm
- net GND: vias 16 -> 5
Other:
- board outline added: 93.5 x 75 mm
- board text added: "${REFERENCE}"
- board text added: "GND"
- board text added: "GPIO"
- board text added: "K"
- board text added: "Line-In (MIC)"
- board text added: "Line-Out (SPK)"
- board text added: "SVXLink MTM5400 interface"
- board text added: "v1.5"
- board text removed: "Isolated SVXLink interface from usb-audio card to MTM5400"
- board text removed: "v1.4"
